Commit message: progress on task 2

File: src/IAS0220_252062IV/urdf/differential_robot.urdf (robot description, URDF)
Before this commit: robot my_robot, 7 links, 6 joints
Links:
- link passive_wheel: geometry visual sphere radius=0.012
Joints:
- joint base_to_head: origin xyz=0.18 0 0.03 rpy=0 0 0 -> xyz=0.15 0 0.05 rpy=0 0 0
- joint base_to_passive_holder: origin xyz=-0.16 0 0 rpy=0 0 0 -> xyz=-0.15 0 0.01 rpy=0 0 0
- joint holder_to_passive_wheel: origin xyz=0 0 -0.035 rpy=0 0 0 -> xyz=0 0 -0.03 rpy=0 0 0

Commit message: task 2 finished

File: src/IAS0220_252062IV/urdf/differential_robot.urdf (robot description, URDF)
Before this commit: robot my_robot, 7 links, 6 joints
Links:
- added link lw_marker; visual box size=0.03 0.03 0.001
- added link rw_marker; visual box size=0.03 0.03 0.001
- link base_link: mass 10 -> None; geometry visual box size=0.33 0.34 0.01
- link left_wheel: geometry visual cylinder length=0.01 radius=0.036
- link passive_wheel: geometry visual sphere radius=0.0105
- link passive_wheel_holder: geometry visual box size=0.02 0.02 0.04
- link right_wheel: geometry visual cylinder length=0.01 radius=0.036
Joints:
- added joint lw_marker_joint: type fixed, parent left_wheel, child lw_marker, origin xyz=0 0 -0.005 rpy=0 0 0
- added joint rw_marker_joint: type fixed, parent right_wheel, child rw_marker, origin xyz=0 0 0.005 rpy=0 0 0
- joint base_to_head: origin xyz=0.15 0 0.05 rpy=0 0 0 -> xyz=0.15 0 0.02 rpy=0 0 0
- joint base_to_left_wheel: axis 0 1 0 -> 0 0 1; origin xyz=0 0.18 0.036 rpy=0 0 0 -> xyz=0 0.175 0 rpy=1.5708 0 0
- joint base_to_passive_holder: origin xyz=-0.15 0 0.01 rpy=0 0 0 -> xyz=0.15 0 -0.008 rpy=0 0 0
- joint base_to_right_wheel: axis 0 1 0 -> 0 0 1; origin xyz=0 -0.18 0.036 rpy=0 0 0 -> xyz=0 -0.175 0 rpy=1.5708 0 0
- joint footprint_to_base: origin xyz=0 0 0 rpy=0 0 0 -> xyz=0 0 0.036 rpy=0 0 0
- joint holder_to_passive_wheel: origin xyz=0 0 -0.03 rpy=0 0 0 -> xyz=0 0 -0.022 rpy=0 0 0

Commit message: task 2.2 almost finished

File: src/IAS0220_252062IV/urdf/differential_robot.urdf (robot description, URDF)
Before this commit: robot my_robot, 9 links, 8 joints
Links:
- removed link base_link
- removed link head_marker
- removed link left_wheel
- removed link lw_marker
- removed link passive_wheel_holder
- removed link right_wheel
- removed link rw_marker
- link passive_wheel: mass None -> 0.01; geometry collision sphere radius=0.0105; visual sphere radius=0.0105
Joints:
- removed joint base_to_head
- removed joint base_to_left_wheel
- removed joint base_to_passive_holder
- removed joint base_to_right_wheel
- removed joint footprint_to_base
- removed joint holder_to_passive_wheel
- removed joint lw_marker_joint
- removed joint rw_marker_joint

Commit message: changed after feedback

File: src/IAS0220_252062IV/urdf/differential_robot.urdf (robot description, URDF)
Before this commit: robot my_robot, 2 links, 0 joints
Links:
- link passive_wheel: geometry collision sphere radius=0.0105; visual sphere radius=0.01
